File: Robonova 1 renewed design/Adafruit PCA9685 rev C/Adafruit PCA9685 rev C.kicad_pcb (KiCad board)
At the start: 2 copper layers, 62.2 x 25.4 mm, 40 parts, among them J1 TERMBLOCK_1X2, Q1 AOD417, U1 PCA9685

Commit message: Global pcb layout sketch and obtained data
Parts:
- added JL1: Conn_01x15_Male, Connector_PinHeader_2.54mm:PinHeader_1x15_P2.54mm_Vertical, F.Cu at (109.2, 77.5)
- added JR1: Conn_01x15_Male, Connector_PinHeader_2.54mm:PinHeader_1x15_P2.54mm_Vertical, F.Cu at (193.0, 78.7)
- added JSensor1: Conn_01x15_Male, Connector_PinHeader_2.54mm:PinHeader_1x15_P2.54mm_Vertical, F.Cu at (129.5, 72.4)
- added LS1: Speaker, Capacitor_THT:CP_Radial_D12.5mm_P7.50mm, F.Cu at (176.5, 80.0)
- added Q2: BC547, Package_TO_SOT_THT:TO-92_Inline, F.Cu at (182.9, 68.6)
- added R1: 1K, Adafruit PCA9685 rev C:0805-NO, F.Cu at (177.5, 68.6)
Connections:
- U1 pad 24: /A5 -> Net-(U1-Pad24)
- U1 pad 3: /A2 -> Net-(U1-Pad3)
- U1 pad 4: /A3 -> Net-(U1-Pad4)
- U1 pad 5: /A4 -> Net-(U1-Pad5)
Routing:
- removed copper zone on B.Cu, net GND
