File: Robonova Updated Controller Board/Robonova Updated Controller Board/16servocontroller_sch.kicad_sch (KiCad schematic)
At the start: 38 parts

Commit message: Removed useless files and added some libraries to kicad
Parts:
- C?: value (none) -> 10uF; footprint (none) -> Adafruit PCA9685 rev C:0805-NO
- C?: value (none) -> CPOL-USE3.5-8; footprint (none) -> Adafruit PCA9685 rev C:E3,5-8
- J?: value (none) -> TERMBLOCK_1X2; footprint (none) -> Adafruit PCA9685 rev C:TERMBLOCK_1X2-3.5MM
- JP? (x2): value (none) -> PINHD-1X6CB; footprint (none) -> Adafruit PCA9685 rev C:1X06-CLEANBIG
- JP? (x4): value (none) -> HEADER-3X04; footprint (none) -> Adafruit PCA9685 rev C:3X04
- LED?: value (none) -> GREEN; footprint (none) -> Adafruit PCA9685 rev C:CHIPLED_0805_NOOUTLINE
- Q?: value (none) -> AOD417; footprint (none) -> Adafruit PCA9685 rev C:TO252
- R? (x16): value (none) -> 220; footprint (none) -> Adafruit PCA9685 rev C:RESPACK_4X0603
- R?: value (none) -> 10K; footprint (none) -> Adafruit PCA9685 rev C:0805-NO
- R? (x4): value (none) -> 10K; footprint (none) -> Adafruit PCA9685 rev C:RESPACK_4X0603
- R?: value (none) -> 470; footprint (none) -> Adafruit PCA9685 rev C:_0805MP
- SJ_A? (x2): value (none) -> SOLDERJUMPERREFLOW_NOPASTE; footprint (none) -> Adafruit PCA9685 rev C:SOLDERJUMPER_REFLOW_NOPASTE
- TP? (x2): value (none) -> TESTPOINTROUND1MM; footprint (none) -> Adafruit PCA9685 rev C:TESTPOINT_ROUND_1MM
- U?: value (none) -> PCA9685; footprint (none) -> Adafruit PCA9685 rev C:TSSOP28
